File: board/Brew_Temperature_Controller.sch (KiCad schematic (older format))
At the start: 12 parts, among them J1 CTBP9358/4, J2 CTB0708/2, J3 Conn_01x02_Male, Q1 IRLU024NPBF, SW1 MCDTS6-1R, SW2 MCDTS6-1R, U1 Nokia_5110_Module

Commit message: Board tweaks and software update
The use of D2 to control the heater was a mistake as it does not
provide PWM, switch to using D3.

The chosen MOSFET was not suitable for driving the heater at full
current and has thus been switched for a more powerful one.

Move the README so that it's more general for the whole project rather
than just the board design and use Markdown.

Add license to source code.

Add features to the software:

- Drive output with PWM
- Utilise screen backlight
- Save set temperature across boots
- Display percentage power output when on
- Test for detached thermistor and turn off output as safety measure
- Allow scrolling of setpoint with long press of buttons
- Log to serial at approx 1Hz

Signed-off-by: Martyn Welch <martyn.welch@collabora.com>
Parts:
- Q1: value IRLU024NPBF -> STP60NF06L
Connections:
- net HEATER: now also A1.18 (D3); no longer A1.17 (D2)
Changed lines of the file:
@@
 P 8800 5150
 F 0 "Q1" H 9004 5196 50  0000 L CNN
-F 1 "IRLU024NPBF" H 9004 5105 50  0000 L CNN
+F 1 "STP60NF06L" H 9004 5105 50  0000 L CNN
 F 2 "Package_TO_SOT_THT:TO-251-3-1EP_Horizontal_TabDown" H 9000 5250 50  0001 C CNN
 F 3 "~" H 8800 5150 50  0001 C CNN
@@
 Wire Wire Line
 	8600 5150 8350 5150
-Text GLabel 5250 2900 0    50   Output ~ 0
+Text GLabel 5250 3000 0    50   Output ~ 0
 HEATER
 $Comp
@@
 	5950 4400 5950 4550
 Wire Wire Line
-	5250 2900 5350 2900
+	5250 3000 5350 3000
 Wire Wire Line
 	6350 3300 6450 3300
